File: V5/PCB/V5PCB.kicad_sch (KiCad schematic)
At the start: 63 parts, among them J1 TYPE_C_6PIN_2MD_073, U1 ESP32-C3-MINI-1-N4, U11 ST-0277D00-052-142, U12 SRV05-4_C558418, U2 FM-3510RGBA-SG, U3 M3406, U4 TS-KG012EV, U5 BMI270, U5 TS-KG012EV, U6 FM-3510RGBA-SG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

Commit message: reorganizing CAD files
Parts:
- U3: value ~ -> IP2312
Changed lines of the file:
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@@
   )
   (symbol (lib_id "CosmicLSM_Symbols:IP2312") (at 118.11 35.56 0) (unit 1)
-    (in_bom yes) (on_board yes) (dnp no) (fields_autoplaced)
-    (property "Reference" "U3" (at 120.3041 43.18 0)
+    (in_bom yes) (on_board yes) (dnp no)
+    (property "Reference" "U3" (at 124.46 44.45 0)
       (effects (font (size 1.27 1.27)) (justify left))
     )
-    (property "Value" "~" (at 118.11 35.56 0)
+    (property "Value" "IP2312" (at 111.76 44.45 0)
       (effects (font (size 1.27 1.27)))
     )
