File: V5/PCB/V5Cattail/V5Cattail.kicad_sch (KiCad schematic)
At the start: 8 parts, among them U11 ST-0277D00-052-142, U12 SRV05-4_C558418, U5 BMI270

Commit message: Overdue backup
Parts:
- removed C8, C9: 100n, Capacitor_SMD:C_0603_1608Metric, symbol CosmicLSM_Symbols:C_Small
- removed R18 (x3): 1k, Resistor_SMD:R_0603_1608Metric, symbol CosmicLSM_Symbols:R_Small
- removed U11: ST-0277D00-052-142, AUDIO-TH_ST-0277D00-052-142:AUDIO-TH_ST-0277D00-052-142, symbol ST-0277D00-052-142:ST-0277D00-052-142
- removed U5: BMI270, Package_LGA:Bosch_LGA-14_3x2.5mm_P0.5mm, symbol CosmicLSM_Symbols:BMI270
- added C1, C2: 100nF, LilypadVR:C_0603_1608Metric, symbol LilypadVR:C_Small
- added J1: TRRS, LilypadVR:AUDIO-TH_ST-0277D00-052-142, symbol LilypadVR:Conn_01x05_Socket
- added U2: BMI270, Package_LGA:Bosch_LGA-14_3x2.5mm_P0.5mm, symbol LilypadVR:BMI270
- U12: footprint SOT-23-6_L2.9-W1.6-P0.95-LS2.8-BL:SOT-23-6_L2.9-W1.6-P0.95-LS2.8-BL -> footprint:SOT-23-6_L2.9-W1.6-P0.95-LS2.8-BL; symbol SRV05-4_C558418:SRV05-4_C558418 -> LilypadVR:SRV05-4_C558418
Connections:
- net +3V3: now also C1.2, C2.1, J1.1 (Pin_1), U2.1 (SDO), U2.12 (CSB), U2.5 (VDDIO), U2.8 (VDD)
- net GND: now also C1.1, C2.2, J1.2 (Pin_2), U2.6 (GNDIO), U2.7 (GND)
- net SCL: now also J1.4 (Pin_4), J1.5 (Pin_5), U2.13 (SCx)
- net SDA: now also J1.3 (Pin_3), U2.14 (SDx)
Other:
- note added: "Power Flags"
- note added: "Resistor layout shown is-- --for proper functionality-- --of short protection."
- note added: "SD0->VDDIO= 0x69"
- moved on the sheet: U12

Commit message: Prototype Model/PCB Updates
Parts:
- removed J1: TRRS, LilypadVR:AUDIO-TH_ST-0277D00-052-142, symbol LilypadVR:Conn_01x05_Socket
- added J1: TRRS, LilypadVR:AUDIO-SMD_PJ-342C, symbol Connector:Conn_01x04_Socket
Connections:
- net +3V3: now also J1.1 (Pin_1)
- net GND: now also J1.2 (Pin_2)
- net SCL: now also J1.4 (Pin_4)
- net SDA: now also J1.3 (Pin_3)
Changed lines of the file:
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@@
-	)
-	(junction
-		(at 111.76 82.55)
-		(diameter 0)
-		(color 0 0 0 0)
 	)
 	(junction
@@
 	(wire
 		(pts
-			(xy 111.76 82.55) (xy 111.76 83.82)
-		)
-		(stroke
-			(width 0)
-			(type default)
-		)
-	)
-	(wire
-		(pts
 			(xy 110.49 73.66) (xy 135.89 73.66)
 		)
@@
 		(pts
 			(xy 135.89 76.2) (xy 135.89 77.47)
-		)
-		(stroke
-			(width 0)
-			(type default)
-		)
-	)
-	(wire
-		(pts
-			(xy 110.49 83.82) (xy 111.76 83.82)
 		)
 		(stroke
@@
 	)
 	(symbol
-		(lib_id "LilypadVR:Conn_01x05_Socket")
-		(at 105.41 78.74 0)
+		(lib_name "GND_2")
+		(lib_id "power:GND")
+		(at 172.72 124.46 0)
+		(unit 1)
+		(exclude_from_sim no)
+		(in_bom yes)
+		(on_board yes)
+		(dnp no)
+		(property "Reference" "#PWR08"
+			(at 172.72 130.81 0)
+			(effects
+				(font
+					(size 1.27 1.27)
+				)
+				(hide yes)
+			)
+		)
+		(property "Value" "GND"
+			(at 172.72 128.27 0)
+			(effects
+				(font
+					(size 1.27 1.27)
+				)
+			)
+		)
+		(property "Footprint" ""
+			(at 172.72 124.46 0)
+			(effects
+				(font
+					(size 1.27 1.27)
+				)
+				(hide yes)
+			)
+		)
+		(property "Datasheet" ""
+			(at 172.72 124.46 0)
+			(effects
+				(font
+					(size 1.27 1.27)
+				)
+				(hide yes)
+			)
+		)
+		(property "Description" "Power symbol creates a global label with name \"GND\" , ground"
+			(at 172.72 124.46 0)
+			(effects
+				(font
+					(size 1.27 1.27)
+				)
+				(hide yes)
+			)
+		)
+		(pin "1"
+		)
+		(instances
+			(project "V5Cattail"
+				(path "/ceb3d75c-aa71-45e1-9bf9-9b36fd8d38cb"
+					(reference "#PWR08")
+					(unit 1)
+				)
+			)
+		)
+	)
+	(symbol
+		(lib_id "LilypadVR:C_Small")
+		(at 184.15 68.58 90)
+		(unit 1)
+		(exclude_from_sim no)
+		(in_bom yes)
+		(on_board yes)
+		(dnp no)
+		(property "Reference" "C2"
+			(at 186.055 66.04 90)
+			(effects
+				(font
+					(size 1.27 1.27)
+				)
+				(justify left)
+			)
+		)
+		(property "Value" "100nF"
+			(at 186.69 71.12 90)
+			(effects
+				(font
+					(size 1.27 1.27)
+				)
+				(justify left)
+			)
+		)
+		(property "Footprint" "LilypadVR:C_0603_1608Metric"
+			(at 184.15 68.58 0)
+			(effects
+				(font
+					(size 1.27 1.27)
+				)
+				(hide yes)
+			)
+		)
+		(property "Datasheet" "~"
+			(at 184.15 68.58 0)
+			(effects
+				(font
+					(size 1.27 1.27)
+				)
+				(hide yes)
+			)
+		)
+		(property "Description" "Unpolarized capacitor, small symbol"
+			(at 184.15 68.58 0)
+			(effects
+				(font
+					(size 1.27 1.27)
+				)
+				(hide yes)
+			)
+		)
+		(property "EXTENDED?" "FALSE"
+			(at 184.15 68.58 0)
+			(effects
+				(font
+					(size 1.27 1.27)
+				)
+				(hide yes)
+			)
+		)
+		(property "MPN" "C14663"
+			(at 184.15 68.58 0)
+			(effects
+				(font
+					(size 1.27 1.27)
+				)
+				(hide yes)
+			)
+		)
+		(pin "1"
+		)
+		(pin "2"
+		)
+		(instances
+			(project "V5Cattail"
+				(path "/ceb3d75c-aa71-45e1-9bf9-9b36fd8d38cb"
+					(reference "C2")
+					(unit 1)
+				)
+			)
+		)
+	)
+	(symbol
+		(lib_id "Connector:Conn_01x04_Socket")
+		(at 105.41 76.2 0)
 		(mirror y)
 		(unit 1)
@@
 		(dnp no)
 		(property "Reference" "J1"
-			(at 104.775 71.12 0)
+			(at 105.156 71.374 0)
 			(effects
 				(font
@@
 		)
 		(property "Value" "TRRS"
-			(at 105.41 86.36 0)
-			(effects
-				(font
-					(size 1.27 1.27)
-				)
-			)
-		)
-		(property "Footprint" "LilypadVR:AUDIO-TH_ST-0277D00-052-142"
-			(at 105.41 78.74 0)
+			(at 105.41 83.82 0)
+			(effects
+				(font
+					(size 1.27 1.27)
+				)
+			)
+		)
+		(property "Footprint" "LilypadVR:AUDIO-SMD_PJ-342C"
+			(at 105.41 76.2 0)
 			(effects
 				(font
@@
 		)
 		(property "Datasheet" "~"
-			(at 105.41 78.74 0)
-			(effects
-				(font
-					(size 1.27 1.27)
-				)
-				(hide yes)
-			)
-		)
-		(property "Description" "Generic connector, single row, 01x05, script generated"
-			(at 105.41 78.74 0)
+			(at 105.41 76.2 0)
+			(effects
+				(font
+					(size 1.27 1.27)
+				)
+				(hide yes)
+			)
+		)
+		(property "Description" "Generic connector, single row, 01x04, script generated"
+			(at 105.41 76.2 0)
 			(effects
 				(font
@@
 		)
 		(property "EXTENDED?" "TRUE"
-			(at 105.41 78.74 0)
-			(effects
-				(font
-					(size 1.27 1.27)
-				)
-				(hide yes)
-			)
-		)
-		(property "MPN" "C2837093"
-			(at 105.41 78.74 0)
-			(effects
-				(font
-					(size 1.27 1.27)
-				)
-				(hide yes)
-			)
+			(at 105.41 76.2 0)
+			(effects
+				(font
+					(size 1.27 1.27)
+				)
+				(hide yes)
+			)
+		)
+		(property "MPN" "C2837091"
+			(at 105.41 76.2 0)
+			(effects
+				(font
+					(size 1.27 1.27)
+				)
+				(hide yes)
+			)
+		)
+		(pin "3"
+		)
+		(pin "1"
 		)
 		(pin "4"
 		)
 		(pin "2"
-		)
-		(pin "1"
-		)
-		(pin "5"
-		)
-		(pin "3"
 		)
 		(instances
@@
 					(unit 1)
 				)
-			)
-		)
-	)
-	(symbol
-		(lib_name "GND_2")
-		(lib_id "power:GND")
-		(at 172.72 124.46 0)
-		(unit 1)
-		(exclude_from_sim no)
-		(in_bom yes)
-		(on_board yes)
-		(dnp no)
-		(property "Reference" "#PWR08"
-			(at 172.72 130.81 0)
-			(effects
-				(font
-					(size 1.27 1.27)
-				)
-				(hide yes)
-			)
-		)
-		(property "Value" "GND"
-			(at 172.72 128.27 0)
-			(effects
-				(font
-					(size 1.27 1.27)
-				)
-			)
-		)
-		(property "Footprint" ""
-			(at 172.72 124.46 0)
-			(effects
-				(font
-					(size 1.27 1.27)
-				)
-				(hide yes)
-			)
-		)
-		(property "Datasheet" ""
-			(at 172.72 124.46 0)
-			(effects
-				(font
-					(size 1.27 1.27)
-				)
-				(hide yes)
-			)
-		)
-		(property "Description" "Power symbol creates a global label with name \"GND\" , ground"
-			(at 172.72 124.46 0)
-			(effects
-				(font
-					(size 1.27 1.27)
-				)
-				(hide yes)
-			)
-		)
-		(pin "1"
-		)
-		(instances
-			(project "V5Cattail"
-				(path "/ceb3d75c-aa71-45e1-9bf9-9b36fd8d38cb"
-					(reference "#PWR08")
-					(unit 1)
-				)
-			)
-		)
-	)
-	(symbol
-		(lib_id "LilypadVR:C_Small")
-		(at 184.15 68.58 90)
-		(unit 1)
-		(exclude_from_sim no)
-		(in_bom yes)
-		(on_board yes)
-		(dnp no)
-		(property "Reference" "C2"
-			(at 186.055 66.04 90)
-			(effects
-				(font
-					(size 1.27 1.27)
-				)
-				(justify left)
-			)
-		)
-		(property "Value" "100nF"
-			(at 186.69 71.12 90)
-			(effects
-				(font
-					(size 1.27 1.27)
-				)
-				(justify left)
-			)
-		)
-		(property "Footprint" "LilypadVR:C_0603_1608Metric"
-			(at 184.15 68.58 0)
-			(effects
-				(font
-					(size 1.27 1.27)
-				)
-				(hide yes)
-			)
-		)
-		(property "Datasheet" "~"
-			(at 184.15 68.58 0)
-			(effects
-				(font
-					(size 1.27 1.27)
-				)
-				(hide yes)
-			)
-		)
-		(property "Description" "Unpolarized capacitor, small symbol"
-			(at 184.15 68.58 0)
-			(effects
-				(font
-					(size 1.27 1.27)
-				)
-				(hide yes)
-			)
-		)
-		(property "EXTENDED?" "FALSE"
-			(at 184.15 68.58 0)
-			(effects
-				(font
-					(size 1.27 1.27)
-				)
-				(hide yes)
-			)
-		)
-		(property "MPN" "C14663"
-			(at 184.15 68.58 0)
-			(effects
-				(font
-					(size 1.27 1.27)
-				)
-				(hide yes)
-			)
-		)
-		(pin "1"
-		)
-		(pin "2"
-		)
-		(instances
-			(project "V5Cattail"
-				(path "/ceb3d75c-aa71-45e1-9bf9-9b36fd8d38cb"
-					(reference "C2")
-					(unit 1)
-				)
